File: RSC-LV3-LVBPS.kicad_sch (KiCad schematic)
At the start: 15 parts, among them J1 Conn_01x02, J2 Molex 43045-0400, J3 Conn_01x02, J4 Conn_01x02, Q1 AO3400A

Commit message: minor layout and silkscreen tweaks
Parts:
- J1, J3, J4: footprint Connector_Molex:Molex_Micro-Fit_3.0_43650-0200_1x02_P3.00mm_Horizontal -> Project_Library:Molex_Micro-Fit_3.0_43650-0200_1x02_P3.00mm_Horizontal_VerticalCompatible
- J2: footprint Connector_Molex:Molex_Micro-Fit_3.0_43045-0400_2x02_P3.00mm_Horizontal -> Project_Library:Molex_Micro-Fit_3.0_43045-0400_2x02_P3.00mm_Horizontal_VerticalCompatible
Changed lines of the file:
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@@
 			)
 		)
-		(property "Footprint" "Connector_Molex:Molex_Micro-Fit_3.0_43650-0200_1x02_P3.00mm_Horizontal"
+		(property "Footprint" "Project_Library:Molex_Micro-Fit_3.0_43650-0200_1x02_P3.00mm_Horizontal_VerticalCompatible"
 			(at 78.74 40.64 0)
 			(hide yes)
@@
 			)
 		)
-		(property "Footprint" "Connector_Molex:Molex_Micro-Fit_3.0_43045-0400_2x02_P3.00mm_Horizontal"
+		(property "Footprint" "Project_Library:Molex_Micro-Fit_3.0_43045-0400_2x02_P3.00mm_Horizontal_VerticalCompatible"
 			(at 148.59 96.52 0)
 			(hide yes)
@@
 			)
 		)
-		(property "Footprint" "Connector_Molex:Molex_Micro-Fit_3.0_43650-0200_1x02_P3.00mm_Horizontal"
+		(property "Footprint" "Project_Library:Molex_Micro-Fit_3.0_43650-0200_1x02_P3.00mm_Horizontal_VerticalCompatible"
 			(at 207.01 130.81 0)
 			(hide yes)
@@
 			)
 		)
-		(property "Footprint" "Connector_Molex:Molex_Micro-Fit_3.0_43650-0200_1x02_P3.00mm_Horizontal"
+		(property "Footprint" "Project_Library:Molex_Micro-Fit_3.0_43650-0200_1x02_P3.00mm_Horizontal_VerticalCompatible"
 			(at 215.9 91.44 0)
 			(hide yes)
