File: Indicator_LED.kicad_sch (KiCad schematic)
At the start: 4 parts

Commit message: r0 final
Parts:
- renumbered D9 to D6
Changed lines of the file:
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@@
 		(dnp no)
 		(fields_autoplaced yes)
-		(property "Reference" "#PWR044"
+		(property "Reference" "#PWR047"
 			(at 128.27 109.22 0)
 			(hide yes)
@@
 			(project "RSC-LV3-LVBPS"
 				(path "/4bbf2fff-9f66-421d-84bf-68d1dcd1e11d/4b8add19-2d3e-4ee3-9fc6-a72eb5b6d291/60bb412c-fe9a-4662-b62c-205cebbf95f7"
-					(reference "#PWR044")
+					(reference "#PWR047")
 					(unit 1)
 				)
 				(path "/4bbf2fff-9f66-421d-84bf-68d1dcd1e11d/4b8add19-2d3e-4ee3-9fc6-a72eb5b6d291/ccdf9a5c-a31a-473f-8738-c18c4e0c4a96"
-					(reference "#PWR045")
+					(reference "#PWR048")
 					(unit 1)
 				)
@@
 		(dnp no)
 		(fields_autoplaced yes)
-		(property "Reference" "D9"
+		(property "Reference" "D6"
 			(at 120.65 76.2 0)
 			(show_name no)
@@
 			(project "RSC-LV3-LVBPS"
 				(path "/4bbf2fff-9f66-421d-84bf-68d1dcd1e11d/4b8add19-2d3e-4ee3-9fc6-a72eb5b6d291/60bb412c-fe9a-4662-b62c-205cebbf95f7"
-					(reference "D9")
+					(reference "D6")
 					(unit 1)
 				)
 				(path "/4bbf2fff-9f66-421d-84bf-68d1dcd1e11d/4b8add19-2d3e-4ee3-9fc6-a72eb5b6d291/ccdf9a5c-a31a-473f-8738-c18c4e0c4a96"
-					(reference "D10")
-					(unit 1)
-				)
+					(reference "D7")
+					(unit 1)
+				)
