File: RSC-LV3-LVBPS.kicad_pcb (KiCad board)
At the start: 2 copper layers, 210 x 60 mm, 122 parts, among them J1 Conn_01x02, J2 Molex 43045-0400, J3 Conn_01x02, J4 Conn_01x02, J5 FTSH-105-01-L-DV-K-A, J6 USB_C_Receptacle_USB2.0_16P, J7 Molex 43650-0500, J8 Molex 43650-0500, K1 SANYOU_SRD_Form_A, K2 SANYOU_SRD_Form_A, Q1 AO3400A, Q2 AO3400A, Q3 AO3400A, U1 INA181A2, U2 INA181A2, U3 STM32G0B1CBTx, U4 TPS54302, U5 TLV74033PDBVR, U6 TLP175A, U7 TJA1051T-3, Y1 32.768 kHz 6pF, Y2 Crystal_GND24

Commit message: minor layout and silkscreen tweaks
Parts:
- added J9: Conn_01x09, Connector_PinHeader_2.54mm:PinHeader_1x09_P2.54mm_Vertical, F.Cu at (101.0, 54.0)
- moved D19 1.75 mm to (98.5, 62.2)
- moved R35 1.75 mm to (98.5, 60.5)
- moved R39 1.25 mm to (131.5, 99.5)
- moved S5 1.25 mm to (126.5, 103.0)
- moved S1 1.00 mm to (202.0, 103.0)
Connections:
- U3 pad 43: unconnected-(U3-PB4-Pad43) -> Net-(J9-Pin_4)
- U3 pad 44: unconnected-(U3-PB5-Pad44) -> Net-(J9-Pin_5)
- U3 pad 45: unconnected-(U3-PB6-Pad45) -> Net-(J9-Pin_6)
- U3 pad 46: unconnected-(U3-PB7-Pad46) -> Net-(J9-Pin_7)
- U3 pad 47: unconnected-(U3-PB8-Pad47) -> Net-(J9-Pin_8)
- U3 pad 48: unconnected-(U3-PB9-Pad48) -> Net-(J9-Pin_9)
Routing:
- net GND: track 936.8 -> 912.8 mm
- net +5V: track 190.1 -> 207.6 mm
- net Net-(J9-Pin_4): track 0.00 -> 17.3 mm
- net Net-(J9-Pin_5): track 0.00 -> 16.5 mm
- net Net-(J9-Pin_6): track 0.00 -> 15.6 mm
- net Net-(J9-Pin_7): track 0.00 -> 14.8 mm
- net Net-(J9-Pin_8): track 0.00 -> 14.0 mm
- net Net-(J9-Pin_9): track 0.00 -> 13.6 mm
- net +3.3V: track 333.5 -> 335.3 mm
- net FDCAN1_RX: track 52.9 -> 51.6 mm
- net FDCAN1_TX: track 60.5 -> 59.3 mm
- net V_SENSE_5: track 40.6 -> 40.0 mm
- net PRIMARY_CAN+: track 51.6 -> 52.1 mm
Other:
- board text added: "PB4"
- board text added: "PB5"
- board text added: "PB6"
- board text added: "PB7"
- board text added: "PB8"
- board text added: "PB9"

Commit message: minor layout and silkscreen tweaks
Parts:
- J1, J3, J4: footprint Connector_Molex:Molex_Micro-Fit_3.0_43650-0200_1x02_P3.00mm_Horizontal -> Project_Library:Molex_Micro-Fit_3.0_43650-0200_1x02_P3.00mm_Horizontal_VerticalCompatible
- J2: footprint Connector_Molex:Molex_Micro-Fit_3.0_43045-0400_2x02_P3.00mm_Horizontal -> Project_Library:Molex_Micro-Fit_3.0_43045-0400_2x02_P3.00mm_Horizontal_VerticalCompatible
Routing:
- net GND: track 912.8 -> 915.2 mm
- net +12V_BAT: track 26.3 -> 28.3 mm

Commit message: r0 final
Parts:
- removed the D11 at (239.2, 73.6)
- removed D16: D_Zener, Diode_SMD:D_SOD-323_HandSoldering
- removed the D3 at (246.9, 84.1)
- removed the D6 at (140.6, 84.2)
- removed the D7 at (153.1, 77.0)
- renumbered D14 to D10, D15 to D11, D17 to D12, D18 to D13, D19 to D14, D20 to D15, D4 to D3, D5 to D4, D8 to D5, D9 to D6, D10 to D7, D12 to D8, D13 to D9, J9 to J7, J7 to J8, J8 to J9
Routing:
- net V_SENSE_12_LOAD: track 76.2 -> 74.0 mm
- net V_SENSE_12_DCDC: track 88.4 -> 86.2 mm
- net V_SENSE_12_BAT: track 181.9 -> 179.7 mm
- net V_SENSE_5: track 40.0 -> 37.9 mm
- net V_SENSE_12: track 5.61 -> 3.45 mm
